File: Assignment/Assignment.kicad_sch (KiCad schematic)
At the start: 115 parts, among them J1 Conn_01x06_Male, J10 Conn_01x04_Male, J11 Conn_01x04_Male, J12 Conn_01x04_Male, J13 Conn_01x03_Male, J14 Conn_02x03_Odd_Even, J15 Conn_02x03_Odd_Even, J16 Conn_02x03_Odd_Even, J17 Conn_02x03_Odd_Even, J18 Conn_01x04_Male, J19 Micro_SD_Card, J2 Conn_01x04_Male, J20 USB_B_Micro, J21 Conn_02x06_Counter_Clockwise, J22 Conn_01x08_Male, J3 Conn_01x04_Male, J4 Conn_02x03_Odd_Even, J5 Conn_02x03_Odd_Even, J6 Conn_02x03_Odd_Even, J7 Conn_02x03_Odd_Even, J8 Conn_01x04_Male, J9 Conn_01x04_Male, Q1 BSS123, SW1 SW_DPST, U1 MIC5233-33, U10 FM25V01, U2 MIC5233-33, U3 MIC5233-33, U4 74LVC2GU04, U5 STM32F407VGTx, U6 HMC5983, U7 MPU-6000, U8 MS5611-01BA, U9 MAX3051, Y1 Resonator

Commit message: added PCB Layout
Parts:
- removed C1: C, symbol Device:C_Polarized
- removed C10, C8, C9: 10u, symbol Device:C_Polarized
- removed C11, C12, C13, C14, C15, C16: 10u, symbol Device:C
- removed C7: 10n, symbol Device:C
- removed SW1: SW_DPST, symbol Switch:SW_DPST
- added C1: 1uF, Capacitor_SMD:C_0402_1005Metric, symbol Device:C
- added SW1: SW_MEC_5G, Button_Switch_SMD:SW_SPST_B3U-1000P-B, symbol Switch:SW_MEC_5G
- 100n1: renamed from 100n; footprint (none) -> Capacitor_SMD:C_0402_1005Metric
- C17, C18, C19, C20, C21, C22, C23, C24, C26, C27, C28: footprint (none) -> Capacitor_SMD:C_0402_1005Metric
- C2, C3: value 10n -> 1uF; footprint (none) -> Capacitor_SMD:C_0402_1005Metric
- C4, C5, C6: value 10n -> 2.2uF; footprint (none) -> Capacitor_SMD:C_0402_1005Metric
- D1, D3, D4, D5, D6: footprint (none) -> LED_SMD:LED_0402_1005Metric
- D2, D7: footprint (none) -> Diode_SMD:SOT65P205X100-3N
- F1: footprint (none) -> Fuse:Fuse_0402_1005Metric
- J1: footprint (none) -> Connector_JST:JST_GH_SM06B-GHS-TB_1x06-1MP_P1.25mm_Horizontal
- J10, J11, J12, J18, J2, J3, J8, J9: footprint (none) -> Connector_JST:JST_GH_SM04B-GHS-TB_1x04-1MP_P1.25mm_Horizontal
- J13: footprint (none) -> Connector_JST:JST_GH_SM03B-GHS-TB_1x03-1MP_P1.25mm_Horizontal
- J14, J15, J16, J17, J4, J5, J6, J7: footprint Connector_Harwin:Harwin_Gecko-G125-MVX0605L1X_2x03_P1.25mm_Vertical -> Connector_PinHeader_2.54mm:PinHeader_2x03_P2.54mm_Vertical
- J19: footprint (none) -> Connector_Card:microSD_HC_Molex_104031-0811
- J20: footprint (none) -> Connector_USB:USB_Micro-B_Wuerth_629105150521_CircularHoles
- J21: footprint (none) -> Connector_PinHeader_2.54mm:PinHeader_2x06_P2.54mm_Vertical
- J22: footprint (none) -> Connector_PinHeader_2.54mm:PinHeader_1x08_P2.54mm_Vertical
- JP1: footprint (none) -> Connector_PinHeader_2.54mm:PinHeader_1x02_P2.54mm_Vertical
- L1: footprint (none) -> Inductor_SMD:L_0402_1005Metric
- R1, R10, R11, R12, R13, R14, R15, R16, R17, R18, R19, R2, R20, R21, R22, R23, R24, R25, R26, R27, R28, R29, R3, R30, R31, R32, R33, R34, R35, R36, R37, R38, R39, R4, R40, R41, R5, R6, R7, R8, R9: footprint (none) -> Resistor_SMD:R_0402_1005Metric
- RN1: footprint (none) -> Resistor_SMD:R_Array_Concave_4x0402
- U1, U2, U3: footprint (none) -> eec:Microchip-SOT23-5LD-PL-1-0-0-MFG
- U10: footprint (none) -> Module:Cypress_Semiconductor-51-85066-0-H-IPC_A
- U4: footprint (none) -> Module:SOT65P210X110-6N
- U6: footprint HMC5983-TR -> Module:HMC5983-TR
- U9: footprint (none) -> Package_SO:SOIC-8_3.9x4.9mm_P1.27mm
- Y1: footprint (none) -> Crystal:Resonator_SMD_Murata_CSTxExxV-3Pin_3.0x1.1mm
Connections:
- net +3V3 is gone; now on net VCC_3: C28.1, J19.4 (VDD), R32.1, R33.2, U10. (WP), U3. (VIN)
- net +5V: now also D2.3 (K), D7.3 (K), J1.1 (Pin_1), J10.1 (Pin_1), J11.1 (Pin_1), J12.1 (Pin_1), J14.3 (Pin_3), J14.4 (Pin_4), J15.3 (Pin_3), J15.4 (Pin_4), J16.3 (Pin_3), J16.4 (Pin_4), J17.3 (Pin_3), J17.4 (Pin_4), J18.4 (Pin_4), J2.2 (Pin_2), J3.1 (Pin_1), J8.1 (Pin_1), J9.1 (Pin_1), R25.1, R30.1, C1.1; no longer C4.1
- net BOOT: now also JP1.1 (A); no longer JP1.2 (B)
- net CURR: now also R39.1; no longer R39.2
- net GND: now also C1.2, SW1.1 (A), SW1.2 (A); no longer C24.1, R34.2, U5.14 (NRST)
- net L_1 inter.: no longer C19.1, L1.2, U5.19 (VDD), U5.22 (VDDA), U5.6 (VBAT)
- net SERVO_POWER: now also D2.1 (A), D2.2 (A)
- net VCC: now also C4.1, JP1.2 (B); no longer C20.1, C23.2, D2.3 (K), D7.3 (K), J1.1 (Pin_1), J10.1 (Pin_1), J11.1 (Pin_1), J12.1 (Pin_1), J14.3 (Pin_3), J14.4 (Pin_4), J15.3 (Pin_3), J15.4 (Pin_4), J16.3 (Pin_3), J16.4 (Pin_4), J17.3 (Pin_3), J17.4 (Pin_4), J18.4 (Pin_4), J2.2 (Pin_2), J3.1 (Pin_1), J8.1 (Pin_1), J9.1 (Pin_1), JP1.1 (A), R25.1, R30.1, R31.1, U2. (VIN), U6. (VDD_IO), U7.13 (VDD)
- net VCC_2: now reaches U2. (VIN)
- net VCC_2: now also C20.1, C23.2, C5.1, R31.1, U6. (VDD_IO), U7.13 (VDD); no longer C6.1
- net at J22.4 (Pin_4): now also R39.2; no longer R39.1
- net VCC_3: now reaches U3. (VIN)
- net VCC_3: now also C6.1
- net V_BAT: no longer names the net of R16.2, R17.2, U5.18 (PC3)
- new net: C19.1, L1.2, U5.19 (VDD), U5.22 (VDDA), U5.6 (VBAT)
- new net NRST: C24.1, R34.2, SW1.3 (B), SW1.4 (B), U5.14 (NRST)
- no-connect marks 20 -> 23
Other:
- note added: "CAN BUS"
- note added: "CAN TRANSCEIVER"
- note added: "COMMUNICATION PROTOCOLS"
- note added: "FLIGHT MANAGEMENT UNIT"
- note added: "I2C BUS"
- note added: "SENSORS"
- note added: "SPI BUS"
- note added: "USART BUS"
- note removed: "ARM POWER INPUT"
- note removed: "CAN PROTOCOL"
- note removed: "I2C"
- note removed: "NAME - JAYESH CHAUDHARY EMAIL - jayeshchaudhary21jan@gmail.com"
- note removed: "SPI PROTOCOL"
- note removed: "USART PROTOCOL"
- moved on the sheet: 100n1, C17, C18, C19, C2, C20, C21, C22, C23, C24, C26, C27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
